File: Renogy_Reader_KiCad/Renogy_Reader.kicad_pcb (KiCad board)
At the start: 2 copper layers, 74.4 x 74 mm, 25 parts, among them J2 Conn_02x06_Odd_Even, J3 RJ45, Q1 2N7000, Q2 2N7000, Q3 2N7000, U1 ESP32-DEVKIT-V1, U4 DS18B20

Commit message: updated kicad
Updated kicad to show errors in DS18B20 pins
Other:
- board text added: "ERROR this needs to be flipped"
Changed lines of the file:
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@@
 		(tags "RJ45")
 		(property "Reference" "J3"
-			(at 4.445 -5 360)
+			(at 4.445 -5 0)
 			(layer "F.SilkS")
 			(effects
@@
 		)
 		(property "Value" "RJ45"
-			(at 4.7244 4.3688 360)
+			(at 4.7244 4.3688 0)
 			(layer "F.Fab")
 			(effects
@@
 		)
 		(fp_text user "${REFERENCE}"
-			(at 4.445 2 360)
+			(at 4.445 2 0)
 			(layer "F.Fab")
 			(effects
@@
 		)
 		(fp_text user "${REFERENCE}"
-			(at 1.27 6.35 360)
+			(at 1.27 6.35 0)
 			(layer "F.Fab")
 			(effects
@@
 		(tags "connector JST EH vertical")
 		(property "Reference" "JOptionalBatteryHeader1"
-			(at 1.25 -4 360)
+			(at 1.25 -4 0)
 			(layer "F.SilkS")
 			(effects
@@
 		)
 		(property "Value" "Conn_01x02"
-			(at 1.25 2.2 360)
+			(at 1.25 2.2 0)
 			(layer "F.Fab")
 			(effects
@@
 		)
 		(fp_text user "${REFERENCE}"
-			(at 1.25 0.3 360)
+			(at 1.25 0.3 0)
 			(layer "F.Fab")
 			(effects
@@
 		)
 	)
+	(gr_text "ERROR this needs to be flipped"
+		(at 168.5036 86.1822 -0)
+		(layer "B.SilkS")
+		(effects
+			(font
+				(size 1.5 1.5)
+				(thickness 0.3)
+				(bold yes)
+			)
+			(justify left bottom)
+		)
+	)
 	(gr_text "Renogy_Reader\nMade by Alex\nIn Colorado\nAugust 2024"
 		(at 189.6364 48.1584 -0)
@@
 	(group ""
 		(members "3cfb4f5a-f335-4be0-9a1c-9145136f1c85" "67c9e37e-7f65-456f-b99d-642935e9b858"
-			"6d06ec00-f52c-4c45-ba5b-0db5cf1736ff" "7b0a8b82-33f6-4704-a8f1-7b13f32fb76d"
-			"a0c5c44d-f610-4e5d-825e-ab73a6829277" "e9fa7b45-234c-435b-8d04-4c63696fe304"
-			"fe081201-df82-4bb3-88cd-7111d3b0833e"
+			"7b0a8b82-33f6-4704-a8f1-7b13f32fb76d" "a0c5c44d-f610-4e5d-825e-ab73a6829277"
+			"e9fa7b45-234c-435b-8d04-4c63696fe304" "fe081201-df82-4bb3-88cd-7111d3b0833e"
 		)
 	)
